File: schematic.sch (EAGLE design)
At the start: 2 parts, among them T1 2N2222, U1 ARGON

Commit message: Add resistor to trigger pin
Connections:
- removed net N$3: T1.B, U1.D7
- new net N$1: U1.D7
- new net N$2: T1.B
Other:
- moved on the sheet: T1
Changed lines of the file:
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@@
 <part name="X_1" library="ngspice-simulation" library_urn="urn:adsk.eagle:library:527439" deviceset="GND" device=""/>
 <part name="+3V1" library="supply1" library_urn="urn:adsk.eagle:library:371" deviceset="+3V3" device=""/>
+<part name="R1" library="docu-dummy" library_urn="urn:adsk.eagle:library:215" deviceset="R" device=""/>
 </parts>
 <sheets>
@@
 <attribute name="NAME" x="27.94" y="59.69" size="1.4224" layer="95" align="top-left"/>
 </instance>
-<instance part="T1" gate="G$1" x="81.28" y="81.28" smashed="yes">
-<attribute name="NAME" x="71.12" y="88.9" size="1.778" layer="95"/>
-<attribute name="VALUE" x="71.12" y="86.36" size="1.778" layer="96"/>
+<instance part="T1" gate="G$1" x="83.82" y="81.28" smashed="yes">
+<attribute name="NAME" x="73.66" y="88.9" size="1.778" layer="95"/>
+<attribute name="VALUE" x="73.66" y="86.36" size="1.778" layer="96"/>
 </instance>
 <instance part="X_1" gate="G$1" x="73.66" y="33.02" smashed="yes"/>
@@
 <attribute name="VALUE" x="12.7" y="114.3" size="1.778" layer="96" rot="R90"/>
 </instance>
+<instance part="R1" gate="G$1" x="66.04" y="81.28" smashed="yes"/>
 </instances>
 <busses>
 </busses>
 <nets>
-<net name="N$3" class="0">
-<segment>
-<pinref part="T1" gate="G$1" pin="B"/>
-<pinref part="U1" gate="U1" pin="D7"/>
-<wire x1="78.74" y1="81.28" x2="50.8" y2="81.28" width="0.1524" layer="91"/>
-</segment>
-</net>
 <net name="AROMGND" class="0">
 <segment>
@@
 <segment>
 <pinref part="T1" gate="G$1" pin="E"/>
-<wire x1="83.82" y1="76.2" x2="106.68" y2="76.2" width="0.1524" layer="91"/>
+<wire x1="86.36" y1="76.2" x2="106.68" y2="76.2" width="0.1524" layer="91"/>
 <junction x="106.68" y="76.2"/>
 <label x="109.22" y="76.2" size="1.778" layer="95"/>
@@
 <segment>
 <pinref part="T1" gate="G$1" pin="C"/>
-<wire x1="83.82" y1="86.36" x2="106.68" y2="86.36" width="0.1524" layer="91"/>
+<wire x1="86.36" y1="86.36" x2="106.68" y2="86.36" width="0.1524" layer="91"/>
 <junction x="106.68" y="86.36"/>
 <label x="109.22" y="86.36" size="1.778" layer="95"/>
@@
 </segment>
 </net>
+<net name="N$1" class="0">
+<segment>
+<pinref part="U1" gate="U1" pin="D7"/>
+<wire x1="50.8" y1="81.28" x2="60.96" y2="81.28" width="0.1524" layer="91"/>
+</segment>
+</net>
+<net name="N$2" class="0">
+<segment>
+<pinref part="T1" gate="G$1" pin="B"/>
+<wire x1="71.12" y1="81.28" x2="81.28" y2="81.28" width="0.1524" layer="91"/>
+</segment>
+</net>
